File: board/board.kicad_pcb (KiCad board)
At the start: 2 copper layers, 21 x 13 mm, 1 part

Commit message: initial
Parts:
- added J1: 011_GPIO, on_edge:on_edge_2x05_host, F.Cu at (185.0, 96.5)
- added J2: 011_GPIO, on_edge:on_edge_2x05_device, F.Cu at (140.0, 96.5)
- added R1: 100k, Resistor_SMD:R_0402_1005Metric, F.Cu at (149.6, 100.1)
- added R2: 100k, Resistor_SMD:R_0402_1005Metric, F.Cu at (154.4, 100.1)
- added R3: 100k, Resistor_SMD:R_0402_1005Metric, F.Cu at (159.3, 100.1)
- added R4: 100k, Resistor_SMD:R_0402_1005Metric, F.Cu at (164.2, 100.1)
- added R5: 100k, Resistor_SMD:R_0402_1005Metric, F.Cu at (169.1, 100.1)
- added R6: 100k, Resistor_SMD:R_0402_1005Metric, F.Cu at (174.0, 100.1)
- added SW1: PTS636 SK25J SMTR LFS, Resistor_SMD:R_2512_6332Metric, F.Cu at (149.6, 95.2)
- added SW2: PTS636 SK25J SMTR LFS, Resistor_SMD:R_2512_6332Metric, F.Cu at (154.4, 95.2)
- added SW3: PTS636 SK25J SMTR LFS, Resistor_SMD:R_2512_6332Metric, F.Cu at (159.3, 95.2)
- added SW4: PTS636 SK25J SMTR LFS, Resistor_SMD:R_2512_6332Metric, F.Cu at (164.2, 95.2)
- added SW5: PTS636 SK25J SMTR LFS, Resistor_SMD:R_2512_6332Metric, F.Cu at (169.1, 95.2)
- added SW6: PTS636 SK25J SMTR LFS, Resistor_SMD:R_2512_6332Metric, F.Cu at (174.0, 95.2)
- LOGO1: moved to B.Cu
- moved LOGO1 13.4 mm to (163.0, 95.8), turned to 180 degrees
Routing:
- net Net-(J1-GPIO4): track 0.00 -> 47.4 mm, vias 0 -> 1
- net Net-(J1-GPIO5): track 0.00 -> 47.3 mm, vias 0 -> 1
- net Net-(J1-GPIO3): track 0.00 -> 46.8 mm
- net Net-(J1-GPIO2): track 0.00 -> 46.3 mm, vias 0 -> 2
- net Net-(J1-GPIO1): track 0.00 -> 45.8 mm, vias 0 -> 2
- net Net-(J1-GPIO0): track 0.00 -> 45.4 mm, vias 0 -> 2
- net Net-(J1-GND-Pad8): track 0.00 -> 43.9 mm
- net Net-(J1-3.3V): track 0.00 -> 41.9 mm, vias 0 -> 2
- net Net-(J1-5V): track 0.00 -> 40.8 mm
- net Net-(J1-GND-Pad1): track 0.00 -> 40.5 mm
Other:
- board size 21 x 13 mm -> 45 x 13 mm
- board text added: "osf.100"
- board text added: "osf.b151.v1.0"
